Commit message: update xacro file

File: holonome_description/robots/robot.urdf.xacro (robot description, xacro)
@@ -133,4 +133,90 @@
     </collision>
   </link>
+  <joint name="rouleau_front5_joint" type="continuous">
+    <parent link="wheel_front"/>
+    <child link="rouleau_front5"/>
+    <origin xyz="-3.8 0 17.31" rpy="0 0 0"/>
+    <axis xyz="0 1 0"/>
+  </joint>
+  <link name="rouleau_front5">
+    <visual>
+      <geometry>
+        <mesh filename="package://holonome_description/meshes/rouleau.stl"/>
+      </geometry>
+      <origin xyz="0 0 0" rpy="0 0 ${pi/2}"/>
+    </visual>
+    <collision>
+      <geometry>
+        <mesh filename="package://holonome_description/meshes/rouleau.stl"/>
+      </geometry>
+      <origin xyz="0 0 0" rpy="0 0 ${pi/2}"/>
+    </collision>
+  </link>
+  <joint name="rouleau_front6_joint" type="continuous">
+    <parent link="wheel_front"/>
+    <child link="rouleau_front6"/>
+    <origin xyz="-3.8 17.31 0" rpy="0 0 0"/>
+    <axis xyz="0 0 1"/>
+  </joint>
+  <link name="rouleau_front6">
+    <visual>
+      <geometry>
+        <mesh filename="package://holonome_description/meshes/rouleau.stl"/>
+      </geometry>
+      <origin xyz="0 0 0" rpy="0 ${pi/2} 0"/>
+    </visual>
+    <collision>
+      <geometry>
+        <mesh filename="package://holonome_description/meshes/rouleau.stl"/>
+      </geometry>
+      <origin xyz="0 0 0" rpy="0 ${pi/2} 0"/>
+    </collision>
+  </link>
+  <joint name="rouleau_front7_joint" type="continuous">
+    <parent link="wheel_front"/>
+    <child link="rouleau_front7"/>
+    <origin xyz="-3.8 0 -17.31" rpy="0 0 0"/>
+    <axis xyz="0 1 0"/>
+  </joint>
+  <link name="rouleau_front7">
+    <visual>
+      <geometry>
+        <mesh filename="package://holonome_description/meshes/rouleau.stl"/>
+      </geometry>
+      <origin xyz="0 0 0" rpy="0 0 ${pi/2}"/>
+    </visual>
+    <collision>
+      <geometry>
+        <mesh filename="package://holonome_description/meshes/rouleau.stl"/>
+      </geometry>
+      <origin xyz="0 0 0" rpy="0 0 ${pi/2}"/>
+    </collision>
+  </link>
+  <joint name="rouleau_front8_joint" type="continuous">
+    <parent link="wheel_front"/>
+    <child link="rouleau_front8"/>
+    <origin xyz="-3.8 -17.31 0" rpy="0 0 0"/>
+    <axis xyz="0 0 1"/>
+  </joint>
+  <link name="rouleau_front8">
+    <visual>
+      <geometry>
+        <mesh filename="package://holonome_description/meshes/rouleau.stl"/>
+      </geometry>
+      <origin xyz="0 0 0" rpy="0 ${pi/2} 0"/>
+    </visual>
+    <collision>
+      <geometry>
+        <mesh filename="package://holonome_description/meshes/rouleau.stl"/>
+      </geometry>
+      <origin xyz="0 0 0" rpy="0 ${pi/2} 0"/>
+    </collision>
+  </link>
+  <joint name="wheel_left_joint" type="continuous">
+    <parent link="base_link"/>
+    <child link="wheel_left"/>
+    <origin xyz="-58.6 101.5 -21.4" rpy="0 0 ${pi*2/3}"/>
+    <axis xyz="${cos(pi*2/3)} ${sin(pi*2/3)} 0"/>
+  </joint>
   <link name="wheel_left">
     <visual>
@@ -138,5 +224,5 @@
         <mesh filename="package://holonome_description/meshes/roue.stl"/>
       </geometry>
-      <origin xyz="0 0 0" rpy="0 0 0"/>
+      <origin xyz="0 0 0" rpy="0 ${pi/2} 0"/>
     </visual>
     <collision>
@@ -144,5 +230,5 @@
         <mesh filename="package://holonome_description/meshes/roue.stl"/>
       </geometry>
-      <origin xyz="-58.6 101.5 -21.4" rpy="0 ${pi/2} ${pi*2/3}"/>
+      <origin xyz="0 0 0" rpy="0 ${pi/2} 0"/>
     </collision>
     <!--
@@ -156,8 +242,168 @@
     -->
   </link>
-  <joint name="wheel_left_joint" type="continuous">
+  <joint name="rouleau_left1_joint" type="continuous">
+    <parent link="wheel_left"/>
+    <child link="rouleau_left1"/>
+    <origin xyz="7.4 12.24 -12.24" rpy="0 0 0"/>
+    <axis xyz="0 1 1"/>
+  </joint>
+  <link name="rouleau_left1">
+    <visual>
+      <geometry>
+        <mesh filename="package://holonome_description/meshes/rouleau.stl"/>
+      </geometry>
+      <origin xyz="0 0 0" rpy="0 ${pi/4} ${-pi/2}"/>
+    </visual>
+    <collision>
+      <geometry>
+        <mesh filename="package://holonome_description/meshes/rouleau.stl"/>
+      </geometry>
+      <origin xyz="0 0 0" rpy="0 ${pi/4} ${-pi/2}"/>
+    </collision>
+  </link>
+  <joint name="rouleau_left2_joint" type="continuous">
+    <parent link="wheel_left"/>
+    <child link="rouleau_left2"/>
+    <origin xyz="7.4 -12.24 -12.24" rpy="0 0 0"/>
+    <axis xyz="0 1 -1"/>
+  </joint>
+  <link name="rouleau_left2">
+    <visual>
+      <geometry>
+        <mesh filename="package://holonome_description/meshes/rouleau.stl"/>
+      </geometry>
+      <origin xyz="0 0 0" rpy="0 ${-pi/4} ${-pi/2}"/>
+    </visual>
+    <collision>
+      <geometry>
+        <mesh filename="package://holonome_description/meshes/rouleau.stl"/>
+      </geometry>
+      <origin xyz="0 0 0" rpy="0 ${-pi/4} ${-pi/2}"/>
+    </collision>
+  </link>
+  <joint name="rouleau_left3_joint" type="continuous">
+    <parent link="wheel_left"/>
+    <child link="rouleau_left3"/>
+    <origin xyz="7.4 -12.24 12.24" rpy="0 0 0"/>
+    <axis xyz="0 1 1"/>
+  </joint>
+  <link name="rouleau_left3">
+    <visual>
+      <geometry>
+        <mesh filename="package://holonome_description/meshes/rouleau.stl"/>
+      </geometry>
+      <origin xyz="0 0 0" rpy="0 ${pi/4} ${-pi/2}"/>
+    </visual>
+    <collision>
+      <geometry>
+        <mesh filename="package://holonome_description/meshes/rouleau.stl"/>
+      </geometry>
+      <origin xyz="0 0 0" rpy="0 ${pi/4} ${-pi/2}"/>
+    </collision>
+  </link>
+  <joint name="rouleau_left4_joint" type="continuous">
+    <parent link="wheel_left"/>
+    <child link="rouleau_left4"/>
+    <origin xyz="7.4 12.24 12.24" rpy="0 0 0"/>
+    <axis xyz="0 1 -1"/>
+  </joint>
+  <link name="rouleau_left4">
+    <visual>
+      <geometry>
+        <mesh filename="package://holonome_description/meshes/rouleau.stl"/>
+      </geometry>
+      <origin xyz="0 0 0" rpy="0 ${-pi/4} ${-pi/2}"/>
+    </visual>
+    <collision>
+      <geometry>
+        <mesh filename="package://holonome_description/meshes/rouleau.stl"/>
+      </geometry>
+      <origin xyz="0 0 0" rpy="0 ${pi/4} ${-pi/2}"/>
+    </collision>
+  </link>
+  <joint name="rouleau_left5_joint" type="continuous">
+    <parent link="wheel_left"/>
+    <child link="rouleau_left5"/>
+    <origin xyz="-3.8 0 17.31" rpy="0 0 0"/>
+    <axis xyz="0 1 0"/>
+  </joint>
+  <link name="rouleau_left5">
+    <visual>
+      <geometry>
+        <mesh filename="package://holonome_description/meshes/rouleau.stl"/>
+      </geometry>
+      <origin xyz="0 0 0" rpy="0 0 ${pi/2}"/>
+    </visual>
+    <collision>
+      <geometry>
+        <mesh filename="package://holonome_description/meshes/rouleau.stl"/>
+      </geometry>
+      <origin xyz="0 0 0" rpy="0 0 ${pi/2}"/>
+    </collision>
+  </link>
+  <joint name="rouleau_left6_joint" type="continuous">
+    <parent link="wheel_left"/>
+    <child link="rouleau_left6"/>
+    <origin xyz="-3.8 17.31 0" rpy="0 0 0"/>
+    <axis xyz="0 0 1"/>
+  </joint>
+  <link name="rouleau_left6">
+    <visual>
+      <geometry>
+        <mesh filename="package://holonome_description/meshes/rouleau.stl"/>
+      </geometry>
+      <origin xyz="0 0 0" rpy="0 ${pi/2} 0"/>
+    </visual>
+    <collision>
+      <geometry>
+        <mesh filename="package://holonome_description/meshes/rouleau.stl"/>
+      </geometry>
+      <origin xyz="0 0 0" rpy="0 ${pi/2} 0"/>
+    </collision>
+  </link>
+  <joint name="rouleau_left7_joint" type="continuous">
+    <parent link="wheel_left"/>
+    <child link="rouleau_left7"/>
+    <origin xyz="-3.8 0 -17.31" rpy="0 0 0"/>
+    <axis xyz="0 1 0"/>
+  </joint>
+  <link name="rouleau_left7">
+    <visual>
+      <geometry>
+        <mesh filename="package://holonome_description/meshes/rouleau.stl"/>
+      </geometry>
+      <origin xyz="0 0 0" rpy="0 0 ${pi/2}"/>
+    </visual>
+    <collision>
+      <geometry>
+        <mesh filename="package://holonome_description/meshes/rouleau.stl"/>
+      </geometry>
+      <origin xyz="0 0 0" rpy="0 0 ${pi/2}"/>
+    </collision>
+  </link>
+  <joint name="rouleau_left8_joint" type="continuous">
+    <parent link="wheel_left"/>
+    <child link="rouleau_left8"/>
+    <origin xyz="-3.8 -17.31 0" rpy="0 0 0"/>
+    <axis xyz="0 0 1"/>
+  </joint>
+  <link name="rouleau_left8">
+    <visual>
+      <geometry>
+        <mesh filename="package://holonome_description/meshes/rouleau.stl"/>
+      </geometry>
+      <origin xyz="0 0 0" rpy="0 ${pi/2} 0"/>
+    </visual>
+    <collision>
+      <geometry>
+        <mesh filename="package://holonome_description/meshes/rouleau.stl"/>
+      </geometry>
+      <origin xyz="0 0 0" rpy="0 ${pi/2} 0"/>
+    </collision>
+  </link>
+  <joint name="wheel_right_joint" type="continuous">
     <parent link="base_link"/>
-    <child link="wheel_left"/>
-    <origin xyz="-58.6 101.5 -21.4" rpy="0 ${pi/2} ${pi*2/3}"/>
+    <child link="wheel_right"/>
+    <origin xyz="-58.6 -101.5 -21.4" rpy="0 0 ${-pi*2/3}"/>
     <axis xyz="${cos(pi*2/3)} ${sin(pi*2/3)} 0"/>
   </joint>
@@ -167,5 +413,5 @@
         <mesh filename="package://holonome_description/meshes/roue.stl"/>
       </geometry>
-      <origin xyz="0 0 0" rpy="0 0 0"/>
+      <origin xyz="0 0 0" rpy="0 ${pi/2} 0"/>
     </visual>
     <collision>
@@ -173,5 +419,5 @@
         <mesh filename="package://holonome_description/meshes/roue.stl"/>
       </geometry>
-      <origin xyz="-58.6 -101.5 -21.4" rpy="0 ${pi/2} ${-pi*2/3}"/>
+      <origin xyz="0 0 0" rpy="0 ${pi/2} 0"/>
     </collision>
     <!--
@@ -185,9 +431,163 @@
     -->
   </link>
-  <joint name="wheel_right_joint" type="continuous">
-    <parent link="base_link"/>
-    <child link="wheel_right"/>
-    <origin xyz="-58.6 -101.5 -21.4" rpy="0 ${pi/2} ${-pi*2/3}"/>
-    <axis xyz="${cos(pi*2/3)} ${sin(pi*2/3)} 0"/>
-  </joint>
+  <joint name="rouleau_right1_joint" type="continuous">
+    <parent link="wheel_right"/>
+    <child link="rouleau_right1"/>
+    <origin xyz="7.4 12.24 -12.24" rpy="0 0 0"/>
+    <axis xyz="0 1 1"/>
+  </joint>
+  <link name="rouleau_right1">
+    <visual>
+      <geometry>
+        <mesh filename="package://holonome_description/meshes/rouleau.stl"/>
+      </geometry>
+      <origin xyz="0 0 0" rpy="0 ${pi/4} ${-pi/2}"/>
+    </visual>
+    <collision>
+      <geometry>
+        <mesh filename="package://holonome_description/meshes/rouleau.stl"/>
+      </geometry>
+      <origin xyz="0 0 0" rpy="0 ${pi/4} ${-pi/2}"/>
+    </collision>
+  </link>
+  <joint name="rouleau_right2_joint" type="continuous">
+    <parent link="wheel_right"/>
+    <child link="rouleau_right2"/>
+    <origin xyz="7.4 -12.24 -12.24" rpy="0 0 0"/>
+    <axis xyz="0 1 -1"/>
+  </joint>
+  <link name="rouleau_right2">
+    <visual>
+      <geometry>
+        <mesh filename="package://holonome_description/meshes/rouleau.stl"/>
+      </geometry>
+      <origin xyz="0 0 0" rpy="0 ${-pi/4} ${-pi/2}"/>
+    </visual>
+    <collision>
+      <geometry>
+        <mesh filename="package://holonome_description/meshes/rouleau.stl"/>
+      </geometry>
+      <origin xyz="0 0 0" rpy="0 ${-pi/4} ${-pi/2}"/>
+    </collision>
+  </link>
+  <joint name="rouleau_right3_joint" type="continuous">
+    <parent link="wheel_right"/>
+    <child link="rouleau_right3"/>
+    <origin xyz="7.4 -12.24 12.24" rpy="0 0 0"/>
+    <axis xyz="0 1 1"/>
+  </joint>
+  <link name="rouleau_right3">
+    <visual>
+      <geometry>
+        <mesh filename="package://holonome_description/meshes/rouleau.stl"/>
+      </geometry>
+      <origin xyz="0 0 0" rpy="0 ${pi/4} ${-pi/2}"/>
+    </visual>
+    <collision>
+      <geometry>
+        <mesh filename="package://holonome_description/meshes/rouleau.stl"/>
+      </geometry>
+      <origin xyz="0 0 0" rpy="0 ${pi/4} ${-pi/2}"/>
+    </collision>
+  </link>
+  <joint name="rouleau_right4_joint" type="continuous">
+    <parent link="wheel_right"/>
+    <child link="rouleau_right4"/>
+    <origin xyz="7.4 12.24 12.24" rpy="0 0 0"/>
+    <axis xyz="0 1 -1"/>
+  </joint>
+  <link name="rouleau_right4">
+    <visual>
+      <geometry>
+        <mesh filename="package://holonome_description/meshes/rouleau.stl"/>
+      </geometry>
+      <origin xyz="0 0 0" rpy="0 ${-pi/4} ${-pi/2}"/>
+    </visual>
+    <collision>
+      <geometry>
+        <mesh filename="package://holonome_description/meshes/rouleau.stl"/>
+      </geometry>
+      <origin xyz="0 0 0" rpy="0 ${pi/4} ${-pi/2}"/>
+    </collision>
+  </link>
+  <joint name="rouleau_right5_joint" type="continuous">
+    <parent link="wheel_right"/>
+    <child link="rouleau_right5"/>
+    <origin xyz="-3.8 0 17.31" rpy="0 0 0"/>
+    <axis xyz="0 1 0"/>
+  </joint>
+  <link name="rouleau_right5">
+    <visual>
+      <geometry>
+        <mesh filename="package://holonome_description/meshes/rouleau.stl"/>
+      </geometry>
+      <origin xyz="0 0 0" rpy="0 0 ${pi/2}"/>
+    </visual>
+    <collision>
+      <geometry>
+        <mesh filename="package://holonome_description/meshes/rouleau.stl"/>
+      </geometry>
+      <origin xyz="0 0 0" rpy="0 0 ${pi/2}"/>
+    </collision>
+  </link>
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
Commit message: Add files via upload

File: holonome_description/robots/robot.urdf.xacro (robot description, xacro)
@@ -1,4 +1,9 @@
 <?xml version="1.0" encoding="utf-8"?>
 <robot name="robot" xmlns:xacro="http://www.ros.org/wiki/xacro">
+  <gazebo>
+    <plugin name="gazebo_ros_control" filename="libgazebo_ros_control.so">
+      <robotNamespace>/omnirobot</robotNamespace>
+    </plugin>
+  </gazebo>
   <link name="base_link">
     <visual>
@@ -591,3 +596,33 @@
     </collision>
   </link>
+  <transmission name="trans_front">
+    <type>transmission_interface/SimpleTransmission</type>
+    <joint name="wheel_front_joint">
+      <hardwareInterface>hardware_interface/VelocityJointInterface</hardwareInterface>
+    </joint>
+    <actuator name="motor_front">
+      <hardwareInterface>hardware_interface/VelocityJointInterface</hardwareInterface>
+      <mechanicalReduction>1</mechanicalReduction>
+    </actuator>
+  </transmission>
+  <transmission name="trans_left">
+    <type>transmission_interface/SimpleTransmission</type>
+    <joint name="wheel_left_joint">
+      <hardwareInterface>hardware_interface/VelocityJointInterface</hardwareInterface>
+    </joint>
+    <actuator name="motor_left">
+      <hardwareInterface>hardware_interface/VelocityJointInterface</hardwareInterface>
+      <mechanicalReduction>1</mechanicalReduction>
+    </actuator>
+  </transmission>
+  <transmission name="trans_right">
+    <type>transmission_interface/SimpleTransmission</type>
+    <joint name="wheel_right_joint">
+      <hardwareInterface>hardware_interface/VelocityJointInterface</hardwareInterface>
+    </joint>
+    <actuator name="motor_right">
+      <hardwareInterface>hardware_interface/VelocityJointInterface</hardwareInterface>
+      <mechanicalReduction>1</mechanicalReduction>
+    </actuator>
+  </transmission>
 </robot>
